Commit message: init

File: roverrobotics_description/urdf/accessories/imu.urdf (robot description, URDF)
Before this commit: robot imu, 1 links, 1 joints
Joints:
- joint imu_to_payload: origin xyz=0 0 0 rpy=0 0 0 -> xyz=-0.045 0 0.08 rpy=0 0 0

File: roverrobotics_description/urdf/miti.urdf (robot description, URDF)
Before this commit: robot rover_miti, 6 links, 5 joints
Links:
- added link 80_20; visual box size=0.025 0.025 0.24; visual box size=0.025 0.025 0.24
- added link gps; visual cylinder length=0.083 radius=0.08
Joints:
- added joint gps_to_payload: type fixed, parent payload_link, child gps, origin xyz=0.135 0 0.09
- added joint payload_to_ouster: type fixed, parent payload_link, child 80_20, origin xyz=-0.12 0 0.17
